File: USB-PD-Trigger-Board.kicad_pcb (KiCad board)
At the start: 2 copper layers, 38 x 29.9 mm, 37 parts, among them J1 USB4056-03-A_REVA2, J2 796638-2, Q1 IRF9358TRPBF, Q2 2N7002, Q3 BSL308PE, U1 CYPD3177-24LQ

Commit message: Testing Kiri
Routing:
- net Net-(D3-K): track 2.22 -> 3.58 mm
- net V3P3: track 51.9 -> 50.9 mm
Changed lines of the file:
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@@
+	)
+	(segment
+		(start 123.9 97.9)
+		(end 121.9 97.9)
+		(width 0.254)
+		(layer "F.Cu")
+		(net 5)
 	)
 	(segment
@@
 	)
 	(segment
-		(start 126.7 105.675)
-		(end 126.7 98.9)
+		(start 126.7 100.7)
+		(end 123.9 97.9)
 		(width 0.254)
 		(layer "F.Cu")
@@
 	)
 	(segment
+		(start 126.7 105.675)
+		(end 126.7 100.7)
+		(width 0.254)
+		(layer "F.Cu")
+		(net 5)
+	)
+	(segment
 		(start 114.2 97.9)
 		(end 114 97.9)
@@
 	)
 	(segment
-		(start 125.7 97.9)
-		(end 121.9 97.9)
-		(width 0.254)
-		(layer "F.Cu")
-		(net 5)
-	)
-	(segment
 		(start 123.1 105.65)
 		(end 124.8 105.65)
@@
 		(start 111.5125 106.7125)
 		(end 112.675 106.7125)
-		(width 0.254)
-		(layer "F.Cu")
-		(net 5)
-	)
-	(segment
-		(start 126.7 98.9)
-		(end 125.7 97.9)
 		(width 0.254)
 		(layer "F.Cu")
@@
 	)
 	(segment
+		(start 131.5 106)
+		(end 130.8125 106)
+		(width 0.2)
+		(layer "F.Cu")
+		(net 7)
+	)
+	(segment
 		(start 130.065 107.435)
 		(end 130.8125 106.6875)
@@
 	)
 	(segment
+		(start 132.605 108.588)
+		(end 132.605 107.105)
+		(width 0.2)
+		(layer "F.Cu")
+		(net 7)
+	)
+	(segment
+		(start 132.605 107.105)
+		(end 131.5 106)
+		(width 0.2)
+		(layer "F.Cu")
+		(net 7)
+	)
+	(segment
 		(start 131.5 104)
 		(end 132.25 104)
@@
 	)
 	(segment
-		(start 132 106)
-		(end 130.8125 106)
-		(width 0.2)
-		(layer "F.Cu")
-		(net 7)
-	)
-	(segment
 		(start 130.8125 106)
 		(end 130.8125 104.6875)
@@
 	)
 	(segment
-		(start 132.605 106.605)
-		(end 132 106)
-		(width 0.2)
-		(layer "F.Cu")
-		(net 7)
-	)
-	(segment
-		(start 132.605 108.588)
-		(end 132.605 106.605)
-		(width 0.2)
-		(layer "F.Cu")
-		(net 7)
-	)
-	(segment
 		(start 126.6125 119.0125)
 		(end 126.6125 120.3)
@@
 	)
 	(segment
-		(start 137.3625 118.075)
+		(start 137.4 118.7)
 		(end 137.4 118.1125)
 		(width 0.2)
@@
 	)
 	(segment
+		(start 135.2 118.7)
+		(end 135.4 118.9)
+		(width 0.2)
+		(layer "F.Cu")
+		(net 9)
+	)
+	(segment
+		(start 137.2 118.9)
+		(end 137.4 118.7)
+		(width 0.2)
+		(layer "F.Cu")
+		(net 9)
+	)
+	(segment
+		(start 135.4 118.9)
+		(end 137.2 118.9)
+		(width 0.2)
+		(layer "F.Cu")
+		(net 9)
+	)
+	(segment
 		(start 135.2 118.075)
-		(end 137.3625 118.075)
-		(width 0.2)
-		(layer "F.Cu")
+		(end 135.2 118.7)
+		(width 0.2)
+		(layer "F.Cu")
