File: USB-PD-Trigger-Board.kicad_pcb (KiCad board)
At the start: 2 copper layers, 38 x 29.9 mm, 37 parts, among them J1 USB4056-03-A_REVA2, J2 796638-2, Q1 IRF9358TRPBF, Q2 2N7002, Q3 BSL308PE, U1 CYPD3177-24LQ

Commit message: Commit to test variant support in PCB as well
Parts:
- R5: value 5.1k_0.1W_0603 -> 2.4k_0.1W_0603

Commit message: Testing Prism Agent
Routing:
- net V3P3: track 50.9 -> 52.3 mm
Changed lines of the file:
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@@
+	)
+	(segment
+		(start 126.3 97.9)
+		(end 121.9 97.9)
+		(width 0.254)
+		(layer "F.Cu")
+		(net "V3P3")
 	)
 	(segment
@@
 	)
 	(segment
-		(start 122.0875 105.6125)
-		(end 122.15 105.675)
-		(width 0.2)
+		(start 126.7 105.675)
+		(end 126.7 98.3)
+		(width 0.254)
 		(layer "F.Cu")
 		(net "V3P3")
 	)
 	(segment
-		(start 123.9 97.9)
-		(end 121.9 97.9)
-		(width 0.254)
+		(start 122.0875 105.6125)
+		(end 122.15 105.675)
+		(width 0.2)
 		(layer "F.Cu")
 		(net "V3P3")
@@
 	)
 	(segment
-		(start 126.7 100.7)
-		(end 123.9 97.9)
+		(start 126.7 98.3)
+		(end 126.3 97.9)
 		(width 0.254)
 		(layer "F.Cu")
@@
 		(width 0.254)
 		(layer "F.Cu")
-		(net "V3P3")
-	)
-	(segment
-		(start 126.7 105.675)
-		(end 126.7 100.7)
-		(width 0.254)
-		(layer "F.Cu")
