File: USB-PD-Trigger-Board.kicad_sch (KiCad schematic)
At the start: 36 parts, among them J1 USB4056-03-A_REVA2, Q1 IRF9358TRPBF, Q2 2N7002, Q3 BSL308PE, U1 CYPD3177-24LQ

Commit message: Testing Kiri
Parts:
- R5: value 5.1k_0.1W_0603 -> 2.4k_0.1W_0603; Manufacturer Part Number RC0603FR-075K1L -> RC0603JR-072K4L; Vendor Part Number 311-5.10KHRDKR-ND -> 311-2.4KGRDKR-ND
Other:
- note added: "Testing Kiri Integration"
Changed lines of the file:
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@@
 		(comment 1 "Krishna Swaroop Dhulipalla")
 	)
+	(text "Testing Kiri Integration"
+		(exclude_from_sim no)
+		(at 142.748 176.022 0)
+		(effects
+			(font
+				(size 1.27 1.27)
+			)
+		)
+	)
 	(junction
 		(at 243.84 77.47)
@@
 	)
 	(junction
+		(at 160.02 181.61)
+		(diameter 0)
+		(color 0 0 0 0)
+	)
+	(junction
 		(at 143.51 163.83)
 		(diameter 0)
@@
 	)
 	(junction
-		(at 160.02 184.15)
-		(diameter 0)
-		(color 0 0 0 0)
-	)
-	(junction
 		(at 168.91 95.25)
 		(diameter 0)
@@
 	(wire
 		(pts
-			(xy 127 184.15) (xy 135.89 184.15)
+			(xy 127 181.61) (xy 135.89 181.61)
 		)
 		(stroke
@@
 	(wire
 		(pts
+			(xy 160.02 181.61) (xy 160.02 171.45)
+		)
+		(stroke
+			(width 0)
+			(type default)
+		)
+	)
+	(wire
+		(pts
 			(xy 176.53 210.82) (xy 176.53 203.2)
 		)
@@
 	(wire
 		(pts
-			(xy 140.97 184.15) (xy 160.02 184.15)
+			(xy 140.97 181.61) (xy 160.02 181.61)
 		)
 		(stroke
@@
 	(wire
 		(pts
-			(xy 160.02 191.77) (xy 160.02 184.15)
-		)
-		(stroke
-			(width 0)
-			(type default)
-		)
-	)
-	(wire
-		(pts
 			(xy 295.91 175.26) (xy 295.91 181.61)
 		)
@@
 	(wire
 		(pts
-			(xy 127 180.34) (xy 127 184.15)
+			(xy 127 180.34) (xy 127 181.61)
 		)
 		(stroke
@@
 	(wire
 		(pts
+			(xy 160.02 181.61) (xy 160.02 191.77)
+		)
+		(stroke
+			(width 0)
+			(type default)
+		)
+	)
+	(wire
+		(pts
 			(xy 146.05 133.35) (xy 90.17 133.35)
 		)
@@
 	(wire
 		(pts
-			(xy 160.02 184.15) (xy 160.02 171.45)
-		)
-		(stroke
-			(width 0)
-			(type default)
-		)
-	)
-	(wire
-		(pts
 			(xy 227.33 171.45) (xy 227.33 173.99)
 		)
@@
 	)
 	(symbol
+		(lib_id "Device:R_Small_US")
+		(at 138.43 181.61 90)
+		(unit 1)
+		(exclude_from_sim no)
+		(in_bom yes)
+		(on_board yes)
+		(dnp no)
+		(property "Reference" "R5"
+			(at 136.398 178.816 90)
+			(effects
+				(font
+					(size 1.27 1.27)
+				)
+				(justify right)
+			)
+		)
+		(property "Value" "2.4k_0.1W_0603"
+			(at 131.826 183.896 90)
+			(effects
+				(font
+					(size 1.27 1.27)
+				)
+				(justify right)
+			)
+		)
+		(property "Footprint" "Resistor_SMD:R_0603_1608Metric_Pad0.98x0.95mm_HandSolder"
+			(at 138.43 181.61 0)
+			(effects
+				(font
+					(size 1.27 1.27)
+				)
+				(hide yes)
+			)
+		)
+		(property "Datasheet" "https://www.yageogroup.com/content/datasheet/asset/file/PYU-RC_GROUP_51_ROHS_L"
+			(at 138.43 181.61 0)
+			(effects
+				(font
+					(size 1.27 1.27)
+				)
+				(hide yes)
+			)
+		)
+		(property "Description" "Resistor, small US symbol"
+			(at 138.43 181.61 0)
+			(effects
+				(font
+					(size 1.27 1.27)
+				)
+				(hide yes)
+			)
+		)
+		(property "Manufacturer" "YAGEO"
+			(at 138.43 181.61 90)
+			(effects
+				(font
+					(size 1.27 1.27)
+				)
+				(hide yes)
+			)
+		)
+		(property "Manufacturer Part Number" "RC0603JR-072K4L"
+			(at 138.43 181.61 90)
+			(effects
+				(font
+					(size 1.27 1.27)
+				)
+				(hide yes)
+			)
+		)
+		(property "Vendor" "DigiKey"
+			(at 138.43 181.61 90)
+			(effects
+				(font
+					(size 1.27 1.27)
+				)
+				(hide yes)
+			)
+		)
+		(property "Vendor Part Number" "311-2.4KGRDKR-ND"
+			(at 138.43 181.61 90)
+			(effects
+				(font
+					(size 1.27 1.27)
+				)
+				(hide yes)
+			)
+		)
+		(pin "2"
+		)
+		(pin "1"
+		)
+		(instances
+			(project "USB-PD-Trigger-Board"
+				(path "/6c5f5d69-1c0b-4294-8a58-8db0ec7d5cdf"
+					(reference "R5")
+					(unit 1)
+				)
+			)
+		)
+	)
+	(symbol
 		(lib_id "Device:C_Small")
 		(at 71.12 82.55 0)
@@
 					(unit 1)
 				)
-			)
-		)
-	)
-	(symbol
-		(lib_id "Device:R_Small_US")
-		(at 138.43 184.15 90)
-		(unit 1)
-		(exclude_from_sim no)
-		(in_bom yes)
-		(on_board yes)
-		(dnp no)
-		(property "Reference" "R5"
-			(at 136.398 181.356 90)
-			(effects
-				(font
-					(size 1.27 1.27)
-				)
-				(justify right)
-			)
-		)
-		(property "Value" "5.1k_0.1W_0603"
-			(at 131.826 186.436 90)
-			(effects
-				(font
-					(size 1.27 1.27)
-				)
-				(justify right)
-			)
-		)
-		(property "Footprint" "Resistor_SMD:R_0603_1608Metric_Pad0.98x0.95mm_HandSolder"
-			(at 138.43 184.15 0)
-			(effects
-				(font
-					(size 1.27 1.27)
-				)
-				(hide yes)
-			)
-		)
-		(property "Datasheet" "https://www.yageogroup.com/content/datasheet/asset/file/PYU-RC_GROUP_51_ROHS_L"
-			(at 138.43 184.15 0)
-			(effects
-				(font
-					(size 1.27 1.27)
-				)
-				(hide yes)
-			)
-		)
-		(property "Description" "Resistor, small US symbol"
-			(at 138.43 184.15 0)
-			(effects
-				(font
-					(size 1.27 1.27)
-				)
-				(hide yes)
-			)
-		)
-		(property "Manufacturer" "YAGEO"
-			(at 138.43 184.15 90)
-			(effects
-				(font
-					(size 1.27 1.27)
-				)
-				(hide yes)
-			)
-		)
-		(property "Manufacturer Part Number" "RC0603FR-075K1L"
-			(at 138.43 184.15 90)
-			(effects
-				(font
-					(size 1.27 1.27)
-				)
-				(hide yes)
-			)
-		)
-		(property "Vendor" "DigiKey"
-			(at 138.43 184.15 90)
-			(effects
-				(font
-					(size 1.27 1.27)
-				)
-				(hide yes)
-			)
-		)
-		(property "Vendor Part Number" "311-5.10KHRDKR-ND"
-			(at 138.43 184.15 90)
-			(effects
-				(font
-					(size 1.27 1.27)
-				)
-				(hide yes)
-			)
-		)
-		(pin "2"
-		)
-		(pin "1"
-		)
-		(instances
-			(project "USB-PD-Trigger-Board"
-				(path "/6c5f5d69-1c0b-4294-8a58-8db0ec7d5cdf"
-					(reference "R5")
-					(unit 1)
-				)
