File: USB-PD-Trigger-Board.kicad_sch (KiCad schematic)
At the start: 36 parts, among them J1 USB4056-03-A_REVA2, Q1 IRF9358TRPBF, Q2 2N7002, Q3 BSL308PE, U1 CYPD3177-24LQ

Commit message: Testing Branching feature in KiCAD-Prism
Parts:
- R10: value 49.9k_0.1W_0603 -> 50k_0.1W_0603
Other:
- note added: "Testing Branching Feature"
