File: USB-PD-Trigger-Board.kicad_sch (KiCad schematic)
At the start: 36 parts, among them J1 USB4056-03-A_REVA2, Q1 IRF9358TRPBF, Q2 2N7002, Q3 BSL308PE, U1 CYPD3177-24LQ

Commit message: DNPed type-C Connector on 20V Variant for testing
Other:
- note added: "Testing Variants"
Changed lines of the file:
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@@
 		)
 	)
+	(text "Testing Variants"
+		(exclude_from_sim no)
+		(at 41.91 65.278 0)
+		(effects
+			(font
+				(size 1.27 1.27)
+			)
+		)
+	)
 	(junction
 		(at 243.84 77.47)
@@
 					(reference "J1")
 					(unit 1)
+					(variant
+						(name "20V")
+						(dnp yes)
+					)
 				)
 			)
