File: USB-PD-Trigger-Board.kicad_sch (KiCad schematic)
At the start: 36 parts, among them J1 USB4056-03-A_REVA2, Q1 IRF9358TRPBF, Q2 2N7002, Q3 BSL308PE, U1 CYPD3177-24LQ

Commit message: Add "Testing Hyperlinks" embedded link for ecad-viewer #454 testing
Working-state commit: KiCad 10 re-saves plus a new root-schematic text
item "Testing Hyperlinks" carrying an embedded hyperlink
((href ...) on its effects) to the ecad-viewer hyperlink PR. Ignore the
editor .history directory.
Other:
- note added: "Testing Hyperlinks"
